Commit message: 10.7.3

File: Agricultural_Bot/ros2_ws/src/agri_robot_description/urdf/xacro/wheel_modules.xacro (robot description, xacro)
@@ -60,5 +60,5 @@
         <child link="f1_wheel_link"/>
         <axis xyz="0 1 0"/>
-        <limit lower="-3.1416" upper="3.1416" effort="20" velocity="2"/>
+        <limit lower="-3.1416" upper="3.1416" effort="20" velocity="8.0"/>
         <dynamics damping="0.1" friction="0.05"/>
       </joint>
@@ -121,5 +121,5 @@
         <child link="f2_wheel_link"/>
         <axis xyz="0 -1 0"/>
-        <limit lower="-3.1416" upper="3.1416" effort="20" velocity="2"/>
+        <limit lower="-3.1416" upper="3.1416" effort="20" velocity="8.0"/>
         <dynamics damping="0.1" friction="0.05"/>
       </joint>
@@ -182,5 +182,5 @@
         <child link="r1_wheel_link"/>
         <axis xyz="0 1 0"/>
-        <limit lower="-3.1416" upper="3.1416" effort="20" velocity="2"/>
+        <limit lower="-3.1416" upper="3.1416" effort="20" velocity="8.0"/>
         <dynamics damping="0.1" friction="0.05"/>
       </joint>
@@ -243,5 +243,5 @@
         <child link="r2_wheel_link"/>
         <axis xyz="0 -1 0"/>
-        <limit lower="-3.1416" upper="3.1416" effort="20" velocity="2"/>
+        <limit lower="-3.1416" upper="3.1416" effort="20" velocity="8.0"/>
         <dynamics damping="0.1" friction="0.05"/>
       </joint>
