Commit message: 10.6.1

File: Agricultural_Bot/ros2_ws/src/agri_robot_description/urdf/robot_pick_robot11.urdf (robot description, URDF)
Before this commit: robot agri_robot, 23 links, 22 joints
Links:
- added link mid360_sensor_frame
Joints:
- added joint mid360_sensor_frame_joint: type fixed, parent mid360_link, child mid360_sensor_frame, origin xyz=0 0 0 rpy=0 0 0
- joint mid360_joint: origin xyz=0 0 0 rpy=0 0 0 -> xyz=0.00340747940546549 0.442350202628433 -0.396759378178018 rpy=0 0 0

File: Agricultural_Bot/ros2_ws/src/agri_robot_description/urdf/xacro/parameters.xacro (robot description, xacro)
@@ -8,3 +8,26 @@
   <xacro:property name="steer_limit" value="3.1416" />
   <xacro:property name="wheel_velocity_limit" value="2.0" />
+  <!--
+    The MID-360 mesh was exported in the assembly (CAD) coordinate system,
+    while its URDF link was previously left at the base_link origin.  Keep
+    this reference in the parent link's CAD-aligned coordinates.  The mesh
+    origins are negated in sensors.xacro so the rendered geometry does not
+    move when the link frame is re-based here.
+    This is the current best reference from the SolidWorks mass properties.
+    Replace it with the measured optical-center offset when the final mount
+    datum is available.
+  -->
+  <xacro:property name="mid360_mount_x" value="0.00340747940546549" />
+  <xacro:property name="mid360_mount_y" value="0.442350202628433" />
+  <xacro:property name="mid360_mount_z" value="-0.396759378178018" />
+  <xacro:property name="mid360_mesh_x" value="-0.00340747940546549" />
+  <xacro:property name="mid360_mesh_y" value="-0.442350202628433" />
+  <xacro:property name="mid360_mesh_z" value="0.396759378178018" />
+  <!-- Offset of the optical frame from the re-based MID-360 body frame. -->
+  <xacro:property name="mid360_sensor_x" value="0" />
+  <xacro:property name="mid360_sensor_y" value="0" />
+  <xacro:property name="mid360_sensor_z" value="0" />
+  <xacro:property name="mid360_sensor_roll" value="0" />
+  <xacro:property name="mid360_sensor_pitch" value="0" />
+  <xacro:property name="mid360_sensor_yaw" value="0" />
 </robot>

File: Agricultural_Bot/ros2_ws/src/agri_robot_description/urdf/xacro/sensors.xacro (robot description, xacro)
@@ -4,10 +4,13 @@
     <link name="mid360_link">
         <inertial>
-          <origin xyz="0.00340747940546549 0.442350202628433 -0.396759378178018" rpy="0 0 0"/>
+          <!-- The re-based link origin is the current CAD mass-property
+               reference, so the inertial offset is intentionally zero. -->
+          <origin xyz="0 0 0" rpy="0 0 0"/>
           <mass value="0.141886777754482"/>
           <inertia ixx="4.507764653165E-05" ixy="5.8921312498008E-08" ixz="8.24694405577648E-09" iyy="6.68381603942182E-05" iyz="-7.01486100567329E-06" izz="4.37585906933259E-05"/>
         </inertial>
         <visual>
-          <origin xyz="0 0 0" rpy="0 0 0"/>
+          <!-- Keep the assembly geometry fixed while moving the link frame. -->
+          <origin xyz="${mid360_mesh_x} ${mid360_mesh_y} ${mid360_mesh_z}" rpy="0 0 0"/>
           <geometry>
             <mesh filename="package://${mesh_package}/meshes/visual/mid360_link.STL"/>
@@ -18,5 +21,5 @@
         </visual>
         <collision>
-          <origin xyz="0 0 0" rpy="0 0 0"/>
+          <origin xyz="${mid360_mesh_x} ${mid360_mesh_y} ${mid360_mesh_z}" rpy="0 0 0"/>
           <geometry>
             <mesh filename="package://${mesh_package}/meshes/visual/mid360_link.STL"/>
@@ -25,8 +28,20 @@
       </link>
     <joint name="mid360_joint" type="fixed">
-        <origin xyz="0 0 0" rpy="0 0 0"/>
+        <!-- Values are expressed in base_link's CAD-aligned coordinates;
+             do not pre-apply the base_footprint CAD-to-ROS rotation. -->
+        <origin xyz="${mid360_mount_x} ${mid360_mount_y} ${mid360_mount_z}" rpy="0 0 0"/>
         <parent link="base_link"/>
         <child link="mid360_link"/>
       </joint>
+    <!-- Explicit sensor frame.  It is coincident with the body frame until
+         the measured optical-center offset and mount tilt are available. -->
+    <link name="mid360_sensor_frame"/>
+    <joint name="mid360_sensor_frame_joint" type="fixed">
+        <origin
+          xyz="${mid360_sensor_x} ${mid360_sensor_y} ${mid360_sensor_z}"
+          rpy="${mid360_sensor_roll} ${mid360_sensor_pitch} ${mid360_sensor_yaw}" />
+        <parent link="mid360_link"/>
+        <child link="mid360_sensor_frame"/>
+    </joint>
     <link name="camera_link">
         <inertial>

Commit message: 10.6.2

File: Agricultural_Bot/ros2_ws/src/agri_robot_description/urdf/robot_pick_robot11.urdf (robot description, URDF)
Before this commit: robot agri_robot, 24 links, 23 joints
Links:
- added link camera_lens_link, mass 0.0387408552979231; collision mesh filename=package://agri_robot_description/meshes/visual/camera_optic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; visual mesh filename=package://agri_robot_description/meshes/visual/camera_optic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
- added link d405_sensor_frame
- link camera_optical_frame: mass 0.0387408552979231 -> None; geometry 
Joints:
- added joint camera_optical_joint: type fixed, parent d405_sensor_frame, child camera_optical_frame, origin xyz=0 0 0 rpy=-1.5707963267948966 0 -1.5707963267948966
- added joint d405_sensor_frame_joint: type fixed, parent camera_lens_link, child d405_sensor_frame, origin xyz=0 -0.00014307690930545467 0.0037672840346891284 rpy=3.141592653589793 1.5328357757419624 1.5707963267948966
- joint camera_option_joint: child camera_optical_frame -> camera_lens_link
- joint mid360_sensor_frame_joint: origin xyz=0 0 0 rpy=0 0 0 -> xyz=3.02793952e-05 0.0166943681 -0.00467974305 rpy=3.141592653589793 -1.3089969389957472 1.5707963267948966

File: Agricultural_Bot/ros2_ws/src/agri_robot_description/urdf/xacro/parameters.xacro (robot description, xacro)
@@ -14,7 +14,7 @@
     origins are negated in sensors.xacro so the rendered geometry does not
     move when the link frame is re-based here.
-    This is the current best reference from the SolidWorks mass properties.
-    Replace it with the measured optical-center offset when the final mount
-    datum is available.
+    The body frame retains the SolidWorks mass-property reference. The
+    separate mid360_sensor_* extrinsic below places the simulation emission
+    origin at the optical dome without changing the inertial/body reference.
   -->
   <xacro:property name="mid360_mount_x" value="0.00340747940546549" />
@@ -24,10 +24,49 @@
   <xacro:property name="mid360_mesh_y" value="-0.442350202628433" />
   <xacro:property name="mid360_mesh_z" value="0.396759378178018" />
-  <!-- Offset of the optical frame from the re-based MID-360 body frame. -->
-  <xacro:property name="mid360_sensor_x" value="0" />
-  <xacro:property name="mid360_sensor_y" value="0" />
-  <xacro:property name="mid360_sensor_z" value="0" />
-  <xacro:property name="mid360_sensor_roll" value="0" />
-  <xacro:property name="mid360_sensor_pitch" value="0" />
-  <xacro:property name="mid360_sensor_yaw" value="0" />
+  <!--
+    CAD-derived simulation emission origin: sphere center fitted to the upper
+    optical dome of mid360_link.STL after removing its existing 15-degree tilt.
+    The fitted radius is 22.0105 mm (radial RMS residual 0.0564 mm). This is a
+    geometric optical-window reference, not a factory-calibrated laser origin.
+    Values below are relative to the re-based body origin in CAD coordinates.
+    In base_footprint the scanning frame has X forward, Y left, Z along the
+    dome axis, with pitch -15 degrees: X=(cos15,0,sin15), Y=(0,1,0),
+    Z=(-sin15,0,cos15). R_body_sensor = R_footprint_body^T * Ry(-15deg).
+    This removes the inherited CAD axes and includes the tilt already present
+    in the mesh; the visual/collision geometry must not be rotated again.
+    Replace only this extrinsic estimate when a measured/factory datum exists.
+  -->
+  <xacro:property name="mid360_sensor_x" value="3.02793952e-05" />
+  <xacro:property name="mid360_sensor_y" value="0.0166943681" />
+  <xacro:property name="mid360_sensor_z" value="-0.00467974305" />
+  <xacro:property name="mid360_sensor_roll" value="3.141592653589793" />
+  <xacro:property name="mid360_sensor_pitch" value="-1.3089969389957472" />
+  <xacro:property name="mid360_sensor_yaw" value="1.5707963267948966" />
+  <!--
+    camera_link.STL is the wrist bracket; camera_optical_frame.STL is the
+    D405 housing, retained on camera_lens_link without changing its assembly
+    pose, visual/collision origin, or inertia. Its front normal is
+    (0, 0.0379514348, -0.999279585): the 2.17498-degree CAD tilt is already
+    in the mesh. Removing that tilt gives a 42.09 x 42 x 23 mm housing and
+    a front-glass plane at z=0.070 mm, opposite the rear M3 mounting holes.
+    The first simulation uses an aligned RGB-D virtual pinhole at the front
+    glass center, 3.7 mm inward (D405 depth-start offset from the datasheet).
+    In the untilted housing it is (0,0,3.770 mm). The CAD omits the two front
+    imagers, so this is an explicit central simulation reference, not the
+    calibrated left-imager origin. The physical left-imager 9 mm offset and
+    measured wrist extrinsics can replace this estimate for hardware use.
+    Reference: RealSense D400 Series Datasheet, October 2025, pages 89-93:
+    https://realsenseai.com/wp-content/uploads/2025/09/Intel-RealSense-D400-Series-Datasheet-October-2025.pdf
+    These values are camera_lens_link -> d405_sensor_frame. Gazebo uses
+    X forward through the front glass, Y left, Z up. The separate optical
+    joint then supplies standard ROS X right, Y down, Z forward axes.
+    Roll pi keeps the front normal unchanged while making image-up follow
+    base_footprint +Z at the arm's zero pose. Roll zero inverted the image.
+  -->
+  <xacro:property name="d405_sensor_x" value="0" />
+  <xacro:property name="d405_sensor_y" value="-0.00014307690930545467" />
+  <xacro:property name="d405_sensor_z" value="0.0037672840346891284" />
+  <xacro:property name="d405_sensor_roll" value="3.141592653589793" />
+  <xacro:property name="d405_sensor_pitch" value="1.5328357757419624" />
+  <xacro:property name="d405_sensor_yaw" value="1.5707963267948966" />
 </robot>

File: Agricultural_Bot/ros2_ws/src/agri_robot_description/urdf/xacro/sensors.xacro (robot description, xacro)
@@ -34,6 +34,7 @@
         <child link="mid360_link"/>
       </joint>
-    <!-- Explicit sensor frame.  It is coincident with the body frame until
-         the measured optical-center offset and mount tilt are available. -->
+    <!-- Gazebo rays and point-cloud headers use this scanning frame, whose
+         origin is the CAD optical-dome center and whose axes include the
+         existing mount tilt. Keep the assembly mesh on mid360_link unchanged. -->
     <link name="mid360_sensor_frame"/>
     <joint name="mid360_sensor_frame_joint" type="fixed">
@@ -71,5 +72,6 @@
         <child link="camera_link"/>
       </joint>
-    <link name="camera_optical_frame">
+    <!-- The CAD camera body is a physical link, not a ROS optical frame. -->
+    <link name="camera_lens_link">
         <inertial>
           <origin xyz="-8.27600293560327E-05 -0.000518418102922302 0.0113997621610378" rpy="0 0 0"/>
@@ -96,4 +98,20 @@
         <origin xyz="-0.017221 -0.0195 0.037803" rpy="-1.5898 0 -1.5708"/>
         <parent link="camera_link"/>
+        <child link="camera_lens_link"/>
+      </joint>
+    <link name="d405_sensor_frame"/>
+    <joint name="d405_sensor_frame_joint" type="fixed">
+        <origin
+          xyz="${d405_sensor_x} ${d405_sensor_y} ${d405_sensor_z}"
+          rpy="${d405_sensor_roll} ${d405_sensor_pitch} ${d405_sensor_yaw}" />
+        <parent link="camera_lens_link"/>
+        <child link="d405_sensor_frame"/>
+      </joint>
+    <!-- Aligned color, depth, and CameraInfo all use this massless standard
+         ROS optical frame: X right, Y down, Z forward. -->
+    <link name="camera_optical_frame"/>
+    <joint name="camera_optical_joint" type="fixed">
+        <origin xyz="0 0 0" rpy="-1.5707963267948966 0 -1.5707963267948966"/>
+        <parent link="d405_sensor_frame"/>
         <child link="camera_optical_frame"/>
       </joint>

File: Agricultural_Bot/sim_ws/src/agri_sim_description/urdf/agri_robot.gazebo.urdf.xacro (robot description, xacro)
@@ -6,5 +6,59 @@
   <xacro:arg name="use_ros2_control" default="$(arg use_control)" />
   <xacro:arg name="controller_config" default="" />
+  <xacro:arg name="use_lidar" default="true" />
+  <xacro:arg name="lidar_mode" default="gpu_lidar" />
+  <xacro:arg name="mid360_frame" default="mid360_sensor_frame" />
+  <xacro:arg name="mid360_topic" default="/mid360" />
+  <xacro:arg name="mid360_rate" default="10.0" />
+  <xacro:arg name="mid360_min_range" default="0.1" />
+  <xacro:arg name="mid360_max_range" default="40.0" />
+  <xacro:arg name="mid360_h_samples" default="1875" />
+  <xacro:arg name="mid360_v_samples" default="32" />
+  <xacro:arg name="mid360_h_min" default="-3.141592653589793" />
+  <xacro:arg name="mid360_h_max" default="3.141592653589793" />
+  <xacro:arg name="mid360_v_min" default="-0.12217304763960307" />
+  <xacro:arg name="mid360_v_max" default="0.9075712110370514" />
+  <xacro:arg name="mid360_resolution" default="0.01" />
+  <xacro:arg name="mid360_noise" default="0.005" />
+  <xacro:arg name="mid360_visualize" default="true" />
+  <xacro:arg name="mid360_preset" default="Livox Mid360" />
+  <xacro:arg name="use_camera" default="true" />
+  <xacro:arg name="d405_frame" default="d405_sensor_frame" />
+  <xacro:arg name="d405_optical_frame" default="camera_optical_frame" />
+  <xacro:arg name="d405_topic" default="/d405" />
+  <xacro:arg name="d405_width" default="848" />
+  <xacro:arg name="d405_height" default="480" />
+  <xacro:arg name="d405_rate" default="30.0" />
+  <xacro:arg name="d405_hfov" default="1.5184364492350666" />
+  <xacro:arg name="d405_fx" default="446.802773119128" />
+  <xacro:arg name="d405_fy" default="432.971461265142" />
+  <xacro:arg name="d405_cx" default="424" />
+  <xacro:arg name="d405_cy" default="240" />
+  <xacro:arg name="d405_color_near" default="0.01" />
+  <xacro:arg name="d405_color_far" default="10.0" />
+  <xacro:arg name="d405_depth_near" default="0.07" />
+  <xacro:arg name="d405_depth_far" default="0.5" />
   <xacro:include filename="$(find agri_robot_description)/urdf/agri_robot.urdf.xacro" />
+  <xacro:include filename="$(find agri_sim_sensors)/urdf/mid360.gazebo.xacro" />
+  <xacro:include filename="$(find agri_sim_sensors)/urdf/d405.gazebo.xacro" />
+  <xacro:if value="$(arg use_lidar)">
+    <xacro:agri_mid360_simulation
+      mode="$(arg lidar_mode)" frame_id="$(arg mid360_frame)" topic="$(arg mid360_topic)"
+      rate="$(arg mid360_rate)" min_range="$(arg mid360_min_range)" max_range="$(arg mid360_max_range)"
+      h_samples="$(arg mid360_h_samples)" v_samples="$(arg mid360_v_samples)"
+      h_min="$(arg mid360_h_min)" h_max="$(arg mid360_h_max)"
+      v_min="$(arg mid360_v_min)" v_max="$(arg mid360_v_max)"
+      resolution="$(arg mid360_resolution)" noise="$(arg mid360_noise)"
+      visualize="$(arg mid360_visualize)" preset="$(arg mid360_preset)" />
+  </xacro:if>
+  <xacro:if value="$(arg use_camera)">
+    <xacro:agri_d405_simulation
+      frame_id="$(arg d405_frame)" optical_frame="$(arg d405_optical_frame)"
+      topic="$(arg d405_topic)" width="$(arg d405_width)" height="$(arg d405_height)"
+      rate="$(arg d405_rate)" hfov="$(arg d405_hfov)"
+      fx="$(arg d405_fx)" fy="$(arg d405_fy)" cx="$(arg d405_cx)" cy="$(arg d405_cy)"
+      color_near="$(arg d405_color_near)" color_far="$(arg d405_color_far)"
+      depth_near="$(arg d405_depth_near)" depth_far="$(arg d405_depth_far)" />
+  </xacro:if>
   <xacro:if value="$(arg use_control)">
     <ros2_control name="GazeboSimSystem" type="system">

Commit message: 10.8.1

File: Agricultural_Bot/ros2_ws/src/agri_robot_description/urdf/robot_pick_robot11.urdf (robot description, URDF)
Before this commit: robot agri_robot, 26 links, 25 joints
Links:
- added link mid360_scan_frame
Joints:
- added joint mid360_scan_frame_joint: type fixed, parent mid360_sensor_frame, child mid360_scan_frame, origin xyz=0 0 0 rpy=0 0.2617993877991494 0
- joint f1_wheel_joint: limit lower=-3.1416 upper=3.1416 effort=20 velocity=2 -> lower=-3.1416 upper=3.1416 effort=20 velocity=8.0
- joint f2_wheel_joint: limit lower=-3.1416 upper=3.1416 effort=20 velocity=2 -> lower=-3.1416 upper=3.1416 effort=20 velocity=8.0
- joint r1_wheel_joint: limit lower=-3.1416 upper=3.1416 effort=20 velocity=2 -> lower=-3.1416 upper=3.1416 effort=20 velocity=8.0
- joint r2_wheel_joint: limit lower=-3.1416 upper=3.1416 effort=20 velocity=2 -> lower=-3.1416 upper=3.1416 effort=20 velocity=8.0

File: Agricultural_Bot/ros2_ws/src/agri_robot_description/urdf/xacro/parameters.xacro (robot description, xacro)
@@ -43,4 +43,7 @@
   <xacro:property name="mid360_sensor_pitch" value="-1.3089969389957472" />
   <xacro:property name="mid360_sensor_yaw" value="1.5707963267948966" />
+  <!-- Navigation uses mid360_scan_frame, whose fixed +15 degree pitch
+       cancels the calibrated sensor-frame -15 degree mount tilt. -->
+  <xacro:property name="mid360_scan_pitch_correction" value="0.2617993877991494" />
   <!--
     camera_link.STL is the wrist bracket; camera_optical_frame.STL is the

File: Agricultural_Bot/ros2_ws/src/agri_robot_description/urdf/xacro/sensors.xacro (robot description, xacro)
@@ -44,4 +44,17 @@
         <parent link="mid360_link"/>
         <child link="mid360_sensor_frame"/>
+    </joint>
+    <!--
+      Navigation projects the 3-D cloud in a horizontal frame.  Keep this
+      frame at exactly the calibrated optical-dome origin; only undo the
+      sensor's -15 degree installation pitch.  The point cloud header remains
+      mid360_sensor_frame and is transformed through TF, so changing a frame
+      name can never silently move the scan origin.
+    -->
+    <link name="mid360_scan_frame"/>
+    <joint name="mid360_scan_frame_joint" type="fixed">
+        <origin xyz="0 0 0" rpy="0 ${mid360_scan_pitch_correction} 0"/>
+        <parent link="mid360_sensor_frame"/>
+        <child link="mid360_scan_frame"/>
     </joint>
     <link name="camera_link">
