Commit message: 10.12.1

File: Agricultural_Bot/ros2_ws/src/agri_robot_description/urdf/agri_robot.urdf.xacro (robot description, xacro)
@@ -7,4 +7,5 @@
        explicitly. Standalone/RViz descriptions retain the mimic relation. -->
   <xacro:arg name="use_ros2_control" default="false" />
+  <xacro:arg name="steering_effort_limit" default="10.0" />
   <xacro:include filename="$(find agri_robot_description)/urdf/xacro/parameters.xacro" />
   <xacro:include filename="$(find agri_robot_description)/urdf/xacro/materials.xacro" />

File: Agricultural_Bot/ros2_ws/src/agri_robot_description/urdf/xacro/wheel_modules.xacro (robot description, xacro)
@@ -30,5 +30,5 @@
         <child link="f1_steer_link"/>
         <axis xyz="0 0 -1"/>
-        <limit lower="-3.1416" upper="3.1416" effort="10" velocity="2"/>
+        <limit lower="-3.1416" upper="3.1416" effort="$(arg steering_effort_limit)" velocity="2"/>
         <dynamics damping="0.1" friction="0.05"/>
       </joint>
@@ -91,5 +91,5 @@
           <child link="f2_steer_link"/>
         <axis xyz="0 0 -1"/>
-        <limit lower="-3.1416" upper="3.1416" effort="10" velocity="2"/>
+        <limit lower="-3.1416" upper="3.1416" effort="$(arg steering_effort_limit)" velocity="2"/>
         <dynamics damping="0.1" friction="0.05"/>
       </joint>
@@ -152,5 +152,5 @@
         <child link="r1_steer_link"/>
         <axis xyz="0 0 -1"/>
-        <limit lower="-3.1416" upper="3.1416" effort="10" velocity="2"/>
+        <limit lower="-3.1416" upper="3.1416" effort="$(arg steering_effort_limit)" velocity="2"/>
         <dynamics damping="0.1" friction="0.05"/>
       </joint>
@@ -213,5 +213,5 @@
         <child link="r2_steer_link"/>
         <axis xyz="0 0 -1"/>
-        <limit lower="-3.1416" upper="3.1416" effort="10" velocity="2"/>
+        <limit lower="-3.1416" upper="3.1416" effort="$(arg steering_effort_limit)" velocity="2"/>
         <dynamics damping="0.1" friction="0.05"/>
       </joint>

File: Agricultural_Bot/sim_ws/src/agri_sim_description/urdf/agri_robot.gazebo.urdf.xacro (robot description, xacro)
@@ -6,4 +6,7 @@
   <xacro:arg name="use_ros2_control" default="$(arg use_control)" />
   <xacro:arg name="controller_config" default="" />
+  <!-- Simulation steering authority for loaded tire contact. The canonical
+       description keeps its original limit; this is not a motor rating. -->
+  <xacro:arg name="steering_effort_limit" default="40.0" />
   <xacro:arg name="use_lidar" default="true" />
   <xacro:arg name="lidar_mode" default="gpu_lidar" />

Commit message: 10.14.1

File: Agricultural_Bot/ros2_ws/src/agri_robot_description/urdf/agri_robot.urdf.xacro (robot description, xacro)
@@ -8,4 +8,6 @@
   <xacro:arg name="use_ros2_control" default="false" />
   <xacro:arg name="steering_effort_limit" default="10.0" />
+  <!-- Optional simulation contact model; canonical CAD collision remains the default. -->
+  <xacro:arg name="wheel_collision_geometry" default="mesh" />
   <xacro:include filename="$(find agri_robot_description)/urdf/xacro/parameters.xacro" />
   <xacro:include filename="$(find agri_robot_description)/urdf/xacro/materials.xacro" />

File: Agricultural_Bot/ros2_ws/src/agri_robot_description/urdf/xacro/gripper.xacro (robot description, xacro)
@@ -38,4 +38,11 @@
         <origin xyz="0 0 0" rpy="0 0 0"/>
       </joint>
+    <link name="grasp_tcp"/>
+    <joint name="grasp_tcp_joint" type="fixed">
+        <parent link="tool0"/>
+        <child link="grasp_tcp"/>
+        <origin xyz="${grasp_tcp_x} ${grasp_tcp_y} ${grasp_tcp_z}"
+                rpy="0 ${grasp_tcp_pitch} 0"/>
+      </joint>
     <link name="gripper_left_finger_link">
         <inertial>
@@ -65,5 +72,6 @@
         <child link="gripper_left_finger_link"/>
         <axis xyz="0 0 1"/>
-        <limit lower="0" upper="0.8" effort="20" velocity="2"/>
+        <limit lower="0" upper="${gripper_finger_stroke}" effort="20"
+               velocity="${gripper_finger_velocity}"/>
         <dynamics damping="0.1" friction="0.05"/>
       </joint>
@@ -98,5 +106,6 @@
           <mimic joint="gripper_left_finger_joint" multiplier="1" offset="0"/>
         </xacro:unless>
-        <limit lower="0" upper="0.8" effort="20" velocity="2"/>
+        <limit lower="0" upper="${gripper_finger_stroke}" effort="20"
+               velocity="${gripper_finger_velocity}"/>
         <dynamics damping="0.1" friction="0.05"/>
       </joint>

File: Agricultural_Bot/ros2_ws/src/agri_robot_description/urdf/xacro/parameters.xacro (robot description, xacro)
@@ -5,7 +5,26 @@
   <xacro:property name="mesh_package" value="$(arg mesh_package)" />
   <xacro:property name="wheel_radius" value="0.127" />
+  <xacro:property name="wheel_width" value="0.100" />
+  <xacro:property name="wheel_collision_geometry" value="$(arg wheel_collision_geometry)" />
+  <!-- Lookup rejects unsupported names instead of silently removing collisions. -->
+  <xacro:property name="wheel_collision_is_cylinder"
+                  value="${dict(mesh=False, cylinder=True)[wheel_collision_geometry]}" />
   <xacro:property name="steer_link_mass" value="15.0" />
   <xacro:property name="steer_limit" value="3.1416" />
   <xacro:property name="wheel_velocity_limit" value="2.0" />
+  <!-- CAD gripper: equal positive finger travel CLOSES the jaws. At q=0
+       the minimum mesh-to-mesh aperture is 74.0815 mm. Limiting each jaw
+       to 35 mm leaves 4.0815 mm clearance, instead of the former 0.8 m
+       limit which made the fingers pass through each other. These are
+       conservative simulation geometry limits, not a hardware stroke rating. -->
+  <xacro:property name="gripper_finger_stroke" value="0.035" />
+  <xacro:property name="gripper_finger_velocity" value="0.04" />
+  <!-- Geometric simulation grasp center between the tapered finger tips,
+       clear of the motor housing. Replace after physical TCP calibration.
+       grasp_tcp +Z points out along gripper_base_link -X; +X is the jaw axis. -->
+  <xacro:property name="grasp_tcp_x" value="-0.18" />
+  <xacro:property name="grasp_tcp_y" value="0.0" />
+  <xacro:property name="grasp_tcp_z" value="0.0" />
+  <xacro:property name="grasp_tcp_pitch" value="-1.5707963267948966" />
   <!--
     The MID-360 mesh was exported in the assembly (CAD) coordinate system,

File: Agricultural_Bot/ros2_ws/src/agri_robot_description/urdf/xacro/wheel_modules.xacro (robot description, xacro)
@@ -1,4 +1,25 @@
 <?xml version="1.0"?>
 <robot xmlns:xacro="http://www.ros.org/wiki/xacro">
+  <xacro:macro name="agri_wheel_collision" params="mesh_file">
+    <collision>
+      <xacro:if value="${wheel_collision_is_cylinder}">
+        <!-- STL radius 0.127 m, width 0.100 m and center (0,0.05,0)
+             before the CAD mesh origin y=-0.05. The cylinder is centered
+             at the wheel link origin with its axis along Y. It encloses
+             the tire chamfers: local X support grows by at most 0.215 mm.
+             Visuals, inertia, joints and navigation footprint are unchanged. -->
+        <origin xyz="0 0 0" rpy="1.5707963267948966 0 0"/>
+        <geometry>
+          <cylinder radius="${wheel_radius}" length="${wheel_width}"/>
+        </geometry>
+      </xacro:if>
+      <xacro:unless value="${wheel_collision_is_cylinder}">
+        <origin xyz="0 -0.05 0" rpy="0 0 0"/>
+        <geometry>
+          <mesh filename="package://${mesh_package}/meshes/visual/${mesh_file}"/>
+        </geometry>
+      </xacro:unless>
+    </collision>
+  </xacro:macro>
   <xacro:macro name="agri_wheel_modules">
     <link name="f1_steer_link">
@@ -48,10 +69,5 @@
           </material>
         </visual>
-        <collision>
-          <origin xyz="0 -0.05 0" rpy="0 0 0"/>
-          <geometry>
-            <mesh filename="package://${mesh_package}/meshes/visual/f1_wheel_link.STL"/>
-          </geometry>
-        </collision>
+        <xacro:agri_wheel_collision mesh_file="f1_wheel_link.STL" />
       </link>
     <joint name="f1_wheel_joint" type="continuous">
@@ -109,10 +125,5 @@
           </material>
         </visual>
-        <collision>
-          <origin xyz="0 -0.05 0" rpy="0 0 0"/>
-          <geometry>
-            <mesh filename="package://${mesh_package}/meshes/visual/f2_wheel_link.STL"/>
-          </geometry>
-        </collision>
+        <xacro:agri_wheel_collision mesh_file="f2_wheel_link.STL" />
       </link>
     <joint name="f2_wheel_joint" type="continuous">
@@ -170,10 +181,5 @@
           </material>
         </visual>
-        <collision>
-          <origin xyz="0 -0.05 0" rpy="0 0 0"/>
-          <geometry>
-            <mesh filename="package://${mesh_package}/meshes/visual/r1_wheel_link.STL"/>
-          </geometry>
-        </collision>
+        <xacro:agri_wheel_collision mesh_file="r1_wheel_link.STL" />
       </link>
     <joint name="r1_wheel_joint" type="continuous">
@@ -231,10 +237,5 @@
           </material>
         </visual>
-        <collision>
-          <origin xyz="0 -0.05 0" rpy="0 0 0"/>
-          <geometry>
-            <mesh filename="package://${mesh_package}/meshes/visual/r2_wheel_link.STL"/>
-          </geometry>
-        </collision>
+        <xacro:agri_wheel_collision mesh_file="r2_wheel_link.STL" />
       </link>
     <joint name="r2_wheel_joint" type="continuous">

File: Agricultural_Bot/sim_ws/src/agri_sim_description/urdf/agri_robot.gazebo.urdf.xacro (robot description, xacro)
@@ -9,5 +9,20 @@
        description keeps its original limit; this is not a motor rating. -->
   <xacro:arg name="steering_effort_limit" default="40.0" />
+  <xacro:arg name="wheel_collision_geometry" default="mesh" />
   <xacro:arg name="use_lidar" default="true" />
+  <xacro:arg name="use_collision_scan" default="false" />
+  <xacro:arg name="collision_scan_frame" default="mid360_sensor_frame" />
+  <xacro:arg name="collision_scan_topic" default="/hard_obstacles" />
+  <xacro:arg name="collision_scan_rate" default="10.0" />
+  <xacro:arg name="collision_scan_min_range" default="0.1" />
+  <xacro:arg name="collision_scan_max_range" default="8.0" />
+  <xacro:arg name="collision_scan_h_samples" default="720" />
+  <xacro:arg name="collision_scan_v_samples" default="16" />
+  <xacro:arg name="collision_scan_h_min" default="-3.141592653589793" />
+  <xacro:arg name="collision_scan_h_max" default="3.141592653589793" />
+  <xacro:arg name="collision_scan_v_min" default="-0.6108652381980153" />
+  <xacro:arg name="collision_scan_v_max" default="0.9075712110370514" />
+  <xacro:arg name="collision_scan_resolution" default="0.01" />
+  <xacro:arg name="collision_scan_noise" default="0.0" />
   <xacro:arg name="lidar_mode" default="gpu_lidar" />
   <xacro:arg name="mid360_frame" default="mid360_sensor_frame" />
@@ -45,4 +60,5 @@
   <xacro:include filename="$(find agri_sim_sensors)/urdf/mid360.gazebo.xacro" />
   <xacro:include filename="$(find agri_sim_sensors)/urdf/d405.gazebo.xacro" />
+  <xacro:include filename="$(find agri_sim_sensors)/urdf/collision_scan.gazebo.xacro" />
   <xacro:if value="$(arg use_lidar)">
     <xacro:agri_mid360_simulation
@@ -54,4 +70,13 @@
       resolution="$(arg mid360_resolution)" noise="$(arg mid360_noise)"
       visualize="$(arg mid360_visualize)" preset="$(arg mid360_preset)" />
+  </xacro:if>
+  <xacro:if value="$(arg use_collision_scan)">
+    <xacro:agri_collision_scan_simulation
+      frame_id="$(arg collision_scan_frame)" topic="$(arg collision_scan_topic)"
+      rate="$(arg collision_scan_rate)" min_range="$(arg collision_scan_min_range)" max_range="$(arg collision_scan_max_range)"
+      h_samples="$(arg collision_scan_h_samples)" v_samples="$(arg collision_scan_v_samples)"
+      h_min="$(arg collision_scan_h_min)" h_max="$(arg collision_scan_h_max)"
+      v_min="$(arg collision_scan_v_min)" v_max="$(arg collision_scan_v_max)"
+      resolution="$(arg collision_scan_resolution)" noise="$(arg collision_scan_noise)" />
   </xacro:if>
   <xacro:if value="$(arg use_camera)">

File: Agricultural_Bot/sim_ws/src/agri_sim_sensors/urdf/d405.gazebo.xacro (robot description, xacro)
@@ -14,4 +14,6 @@
         <always_on>true</always_on>
         <camera>
+          <!-- Preserve normal scene appearance; exclude hidden stem proxies. -->
+          <visibility_mask>268435455</visibility_mask>
           <optical_frame_id>${optical_frame}</optical_frame_id>
           <horizontal_fov>${hfov}</horizontal_fov>

File: Agricultural_Bot/sim_ws/src/agri_sim_sensors/urdf/mid360.gazebo.xacro (robot description, xacro)
@@ -19,4 +19,7 @@
           <visualize>${visualize}</visualize>
           <lidar>
+            <!-- 0x0FFFFFFF: retain the visible plant for localization, but
+                 hide the simulation-only 0x20000000 hard-obstacle proxies. -->
+            <visibility_mask>268435455</visibility_mask>
             <scan>
               <horizontal>

Commit message: 10.14.2

File: Agricultural_Bot/ros2_ws/src/agri_robot_description/urdf/agri_robot.urdf.xacro (robot description, xacro)
@@ -7,4 +7,7 @@
        explicitly. Standalone/RViz descriptions retain the mimic relation. -->
   <xacro:arg name="use_ros2_control" default="false" />
+  <!-- Gazebo may provide a tiny numerical margin at the open-finger stop.
+       The canonical mechanical lower limit remains zero. -->
+  <xacro:arg name="gripper_joint_lower_limit" default="0.0" />
   <xacro:arg name="steering_effort_limit" default="10.0" />
   <!-- Optional simulation contact model; canonical CAD collision remains the default. -->

File: Agricultural_Bot/ros2_ws/src/agri_robot_description/urdf/xacro/gripper.xacro (robot description, xacro)
@@ -72,5 +72,5 @@
         <child link="gripper_left_finger_link"/>
         <axis xyz="0 0 1"/>
-        <limit lower="0" upper="${gripper_finger_stroke}" effort="20"
+        <limit lower="$(arg gripper_joint_lower_limit)" upper="${gripper_finger_stroke}" effort="20"
                velocity="${gripper_finger_velocity}"/>
         <dynamics damping="0.1" friction="0.05"/>
@@ -106,5 +106,5 @@
           <mimic joint="gripper_left_finger_joint" multiplier="1" offset="0"/>
         </xacro:unless>
-        <limit lower="0" upper="${gripper_finger_stroke}" effort="20"
+        <limit lower="$(arg gripper_joint_lower_limit)" upper="${gripper_finger_stroke}" effort="20"
                velocity="${gripper_finger_velocity}"/>
         <dynamics damping="0.1" friction="0.05"/>

File: Agricultural_Bot/sim_ws/src/agri_sim_description/urdf/agri_robot.gazebo.urdf.xacro (robot description, xacro)
@@ -5,4 +5,8 @@
   <xacro:arg name="use_control" default="false" />
   <xacro:arg name="use_ros2_control" default="$(arg use_control)" />
+  <!-- DART 6.13 servo control skips driving q below its lower limit, even
+       for floating-point undershoot. Keep the commanded open position zero
+       inside the simulated range; this 1 um margin changes fingers only. -->
+  <xacro:arg name="gripper_joint_lower_limit" default="-0.000001" />
   <xacro:arg name="controller_config" default="" />
   <!-- Simulation steering authority for loaded tire contact. The canonical
